Commit message: Fix launch description

File: nanosaur_description/urdf/nanosaur.urdf (robot description, URDF)
Before this commit: robot nanosaur, 1 links, 0 joints
Links:
- added link body; visual mesh filename=package://nanosaur_description/meshes/base_rear.stl scale=0.001 0.001 0.001
- added link right_leg; visual box size=0.6 0.1 0.2
- link base_link: geometry 
Joints:
- added joint base_link: type fixed, parent base_link, child body
- added joint base_to_right_leg: type fixed, parent base_link, child right_leg
