Commit message: Improve NanoSaur URDF

File: nanosaur_description/urdf/head.urdf.xacro (robot description, xacro)
@@ -40,5 +40,5 @@
         </link>
         <joint name="camera_joint" type="fixed">
-            <origin xyz="0.010 0 0.0275" rpy="0 ${M_PI/2 - cam_angle * M_PI/180} 0" />
+            <origin xyz="0.010 0 0.0250" rpy="0 ${M_PI/2 - cam_angle * M_PI/180} 0" />
             <parent link="cover"/>
             <child link="camera_board"/>
@@ -46,9 +46,15 @@
         <link name="camera_board">
             <visual>
-                <origin xyz="0 0 0" rpy="0 0 ${M_PI}" />
+                <origin xyz="-0.0025 0 0" rpy="0 0 ${M_PI}" />
                 <geometry><mesh filename="${path_meshes}/parts/rasp_camera.stl"/></geometry>
-                <material name="Black" />
+                <material name="Grey" />
             </visual>
         </link>
+        <joint name="camera_optical_joint" type="fixed">
+            <origin xyz="0 0 0.005" rpy="0 0 -${M_PI/2}"/>
+            <parent link="camera_board"/>
+            <child link="camera_optical_frame"/>
+        </joint>
+        <link name="camera_optical_frame"/>
     </xacro:macro>
 </robot>

File: nanosaur_description/urdf/track.urdf.xacro (robot description, xacro)
@@ -21,7 +21,8 @@
             </visual>
         </link>
-        <joint name="sprocket_${type}_joint" type="fixed">
+        <joint name="sprocket_${type}_joint" type="continuous">
             <parent link="motor_${type}"/>
             <child link="sprocket_${type}"/>
+            <axis xyz="0 0 ${-1 * orientation}" />
         </joint>
         <link name="sprocket_${type}">
@@ -31,9 +32,18 @@
                 <material name="Black" />
             </visual>
+            <!-- Collision cylinder -->
+            <collision>
+                <origin xyz="0 0 0" rpy="0 0 0" />
+                <geometry><cylinder length="0.015" radius="0.0105"/></geometry>
+                <material name="Black" />
+            </collision>
         </link>
-        <joint name="wheel_${type}_joint" type="fixed">
+        <joint name="wheel_${type}_joint" type="continuous">
             <origin xyz="-0.099 0 0" rpy="0 0 0" />
             <parent link="motor_${type}"/>
             <child link="wheel_${type}"/>
+            <axis xyz="0 0 ${-1 * orientation}" />
+            <!-- Passive sprocket rotate automatically according to the status of the active one -->
+            <mimic joint="sprocket_${type}_joint" multiplier="1" offset="0"/>
         </joint>
         <link name="wheel_${type}">
@@ -43,4 +53,10 @@
                 <material name="Black" />
             </visual>
+            <!-- Collision cylinder -->
+            <collision>
+                <origin xyz="0 0 0" rpy="0 0 0" />
+                <geometry><cylinder length="0.015" radius="0.0105"/></geometry>
+                <material name="Black" />
+            </collision>
         </link>
         <joint name="track_${type}_joint" type="fixed">

Commit message: Fix body for power banks with size max 66x94x24 mm

File: nanosaur_description/urdf/head.urdf.xacro (robot description, xacro)
@@ -5,5 +5,5 @@
     <xacro:macro name="head">
         <joint name="cover_joint" type="fixed">
-            <origin xyz="0.06 0 -0.025" rpy="0 0 0" />
+            <origin xyz="0.06 0 -0.026" rpy="0 0 0" />
             <parent link="base_front"/>
             <child link="cover"/>
