Commit message: Add read urdf radius and wheel_distance

File: nanosaur_description/urdf/track.urdf.xacro (robot description, xacro)
@@ -1,5 +1,5 @@
 <?xml version="1.0"?>
 <robot name="nanosaur_track" xmlns:xacro="http://ros.org/wiki/xacro">
-    <xacro:macro name="track" params="type">
+    <xacro:macro name="track" params="type parent radius">
         <!-- Define orientation -->
         <xacro:if value="${type == 'left'}">
@@ -9,18 +9,7 @@
             <xacro:property name="orientation" value="1"/>
         </xacro:if>
-        <joint name="motor_${type}_joint" type="fixed">
-            <origin xyz="0.053 ${orientation * -0.043} -0.015" rpy="${orientation * M_PI/2} 0 0" />
-            <parent link="base_front"/>
-            <child link="motor_${type}"/>
-        </joint>
-        <link name="motor_${type}">
-            <visual>
-                <origin xyz="0 0 -0.031" rpy="0 0 -${M_PI/2}" />
-                <geometry><mesh filename="${path_meshes}/parts/Pololu-Micro-Metal-Gearmotor.stl"/></geometry>
-                <material name="Gold" />
-            </visual>
-        </link>
         <joint name="sprocket_${type}_joint" type="continuous">
-            <parent link="motor_${type}"/>
+            <origin xyz="0.053 ${orientation * -0.043} 0.015" rpy="${orientation * M_PI/2} 0 0" />
+            <parent link="${parent}"/>
             <child link="sprocket_${type}"/>
             <axis xyz="0 0 ${-1 * orientation}" />
@@ -35,7 +24,19 @@
             <collision>
                 <origin xyz="0 0 0" rpy="0 0 0" />
-                <geometry><cylinder length="0.015" radius="0.0105"/></geometry>
+                <geometry><cylinder length="0.015" radius="${radius}"/></geometry>
                 <material name="Black" />
             </collision>
+        </link>
+        <joint name="motor_${type}_joint" type="fixed">
+            <origin xyz="0.053 ${orientation * -0.043} 0.015" rpy="${orientation * M_PI/2} 0 0" />
+            <parent link="${parent}"/>
+            <child link="motor_${type}"/>
+        </joint>
+        <link name="motor_${type}">
+            <visual>
+                <origin xyz="0 0 -0.031" rpy="0 0 -${M_PI/2}" />
+                <geometry><mesh filename="${path_meshes}/parts/Pololu-Micro-Metal-Gearmotor.stl"/></geometry>
+                <material name="Gold" />
+            </visual>
         </link>
         <joint name="wheel_${type}_joint" type="continuous">
@@ -56,5 +57,5 @@
             <collision>
                 <origin xyz="0 0 0" rpy="0 0 0" />
-                <geometry><cylinder length="0.015" radius="0.0105"/></geometry>
+                <geometry><cylinder length="0.015" radius="${radius}"/></geometry>
                 <material name="Black" />
             </collision>

Commit message: Added simulation option

File: nanosaur_description/urdf/track.urdf.xacro (robot description, xacro)
@@ -12,9 +12,10 @@
         <xacro:if value="${mimic_enable}">
             <xacro:property name="mimic_type" value="continuous"/>
+            <xacro:property name="radius_wheel" value="${radius}"/>
         </xacro:if>
         <xacro:unless value="${mimic_enable}">
             <xacro:property name="mimic_type" value="fixed"/>
+            <xacro:property name="radius_wheel" value="${radius-0.005}"/>
         </xacro:unless>
-        <xacro:property name="radius_wheel" value="${radius}"/>
         <joint name="sprocket_${type}_joint" type="continuous">
             <xacro:if value="${diff_drive_emulation}">

Commit message: Improve xacro for Isaac SIM

File: nanosaur_description/urdf/track.urdf.xacro (robot description, xacro)
@@ -12,10 +12,9 @@
         <xacro:if value="${mimic_enable}">
             <xacro:property name="mimic_type" value="continuous"/>
-            <xacro:property name="radius_wheel" value="${radius}"/>
         </xacro:if>
         <xacro:unless value="${mimic_enable}">
             <xacro:property name="mimic_type" value="fixed"/>
-            <xacro:property name="radius_wheel" value="${radius-0.005}"/>
         </xacro:unless>
+        <xacro:property name="radius_wheel" value="${radius}"/>
         <joint name="sprocket_${type}_joint" type="continuous">
             <xacro:if value="${diff_drive_emulation}">
