Commit message: NanoSaur URDF all parts

File: nanosaur_description/urdf/flap.urdf.xacro (robot description, xacro)
@@ -25,4 +25,15 @@
             </visual>
         </link>
+        <joint name="board_expansion_joint" type="fixed">
+            <parent link="flap_bottom"/>
+            <child link="board_expansion"/>
+        </joint>
+        <link name="board_expansion">
+            <visual>
+                <origin xyz="-0.0017 0 0.019" rpy="0 0 0" />
+                <geometry><mesh filename="${path_meshes}/parts/board_expansion.stl"/></geometry>
+                <material name="GunMetalGrey" />
+            </visual>
+        </link>
     </xacro:macro>
 </robot>

File: nanosaur_description/urdf/head.urdf.xacro (robot description, xacro)
@@ -1,4 +1,6 @@
 <?xml version="1.0"?>
 <robot name="nanosaur_head" xmlns:xacro="http://ros.org/wiki/xacro">
+    <xacro:property name="cam_angle" value="5"/>
+    <xacro:property name="display_angle" value="70.6"/>
     <xacro:macro name="head">
         <joint name="cover_joint" type="fixed">
@@ -13,4 +15,40 @@
             </visual>
         </link>
+        <joint name="display_left_joint" type="fixed">
+            <origin xyz="-0.017 0.0244 0.052" rpy="0 ${M_PI/2 - display_angle * M_PI/180} 0" />
+            <parent link="cover"/>
+            <child link="display_left"/>
+        </joint>
+        <link name="display_left">
+            <visual>
+                <origin xyz="0 0 0" rpy="0 0 ${M_PI/2}" />
+                <geometry><mesh filename="${path_meshes}/parts/OLED_Module.stl"/></geometry>
+                <material name="Black" />
+            </visual>
+        </link>
+        <joint name="display_right_joint" type="fixed">
+            <origin xyz="-0.017 -0.0244 0.052" rpy="0 ${M_PI/2 - display_angle * M_PI/180} 0" />
+            <parent link="cover"/>
+            <child link="display_right"/>
+        </joint>
+        <link name="display_right">
+            <visual>
+                <origin xyz="0 0 0" rpy="0 0 ${M_PI/2}" />
+                <geometry><mesh filename="${path_meshes}/parts/OLED_Module.stl"/></geometry>
+                <material name="Black" />
+            </visual>
+        </link>
+        <joint name="camera_joint" type="fixed">
+            <origin xyz="0.010 0 0.0275" rpy="0 ${M_PI/2 - cam_angle * M_PI/180} 0" />
+            <parent link="cover"/>
+            <child link="camera_board"/>
+        </joint>
+        <link name="camera_board">
+            <visual>
+                <origin xyz="0 0 0" rpy="0 0 ${M_PI}" />
+                <geometry><mesh filename="${path_meshes}/parts/rasp_camera.stl"/></geometry>
+                <material name="Black" />
+            </visual>
+        </link>
     </xacro:macro>
 </robot>

Commit message: Update all STL files

File: nanosaur_description/urdf/flap.urdf.xacro (robot description, xacro)
@@ -9,5 +9,6 @@
         <link name="flap_bottom">
             <visual>
-                <origin xyz="-0.0161 0 0.009" rpy="0 0 0" />
+                <!--<origin xyz="-0.0161 0 0.009" rpy="0 0 0" />-->
+                <origin xyz="0.0068 0 0.0175" rpy="0 0 0" />
                 <geometry><mesh filename="${path_meshes}/flap_bottom.stl" scale="0.001 0.001 0.001"/></geometry>
                 <material name="Green" />
@@ -20,5 +21,6 @@
         <link name="flap_top">
             <visual>
-                <origin xyz="-0.0161 0 0.009" rpy="0 0 0" />
+                <!--<origin xyz="-0.0161 0 0.009" rpy="0 0 0" />-->
+                <origin xyz="0.0068 0 0.0175" rpy="0 0 0" />
                 <geometry><mesh filename="${path_meshes}/flap_top.stl" scale="0.001 0.001 0.001"/></geometry>
                 <material name="Green" />
@@ -31,6 +33,7 @@
         <link name="board_expansion">
             <visual>
-                <origin xyz="-0.0017 0 0.019" rpy="0 0 0" />
-                <geometry><mesh filename="${path_meshes}/parts/board_expansion.stl"/></geometry>
+                <!--<origin xyz="-0.0017 0 0.019" rpy="0 0 0" />-->
+                <origin xyz="-0.002 0.0005 0.017" rpy="0 0 0" />
+                <geometry><mesh filename="${path_meshes}/parts/nanosaur-exp-board.stl"/></geometry>
                 <material name="GunMetalGrey" />
             </visual>

File: nanosaur_description/urdf/head.urdf.xacro (robot description, xacro)
@@ -16,5 +16,5 @@
         </link>
         <joint name="display_left_joint" type="fixed">
-            <origin xyz="-0.017 0.0244 0.052" rpy="0 ${M_PI/2 - display_angle * M_PI/180} 0" />
+            <origin xyz="-0.024 0.0242 0.060" rpy="0 ${M_PI/2 - display_angle * M_PI/180} 0" />
             <parent link="cover"/>
             <child link="display_left"/>
@@ -28,5 +28,5 @@
         </link>
         <joint name="display_right_joint" type="fixed">
-            <origin xyz="-0.017 -0.0244 0.052" rpy="0 ${M_PI/2 - display_angle * M_PI/180} 0" />
+            <origin xyz="-0.024 -0.0242 0.060" rpy="0 ${M_PI/2 - display_angle * M_PI/180} 0" />
             <parent link="cover"/>
             <child link="display_right"/>
@@ -40,5 +40,5 @@
         </link>
         <joint name="camera_joint" type="fixed">
-            <origin xyz="0.010 0 0.0250" rpy="0 ${M_PI/2 - cam_angle * M_PI/180} 0" />
+            <origin xyz="0.013 0 0.0280" rpy="0 ${M_PI/2 - cam_angle * M_PI/180} 0" />
             <parent link="cover"/>
             <child link="camera_board"/>

Commit message: New nanosaur urdf description for gazebo simulation

File: nanosaur_description/urdf/flap.urdf.xacro (robot description, xacro)
@@ -2,4 +2,13 @@
 <robot name="nanosaur_flap" xmlns:xacro="http://ros.org/wiki/xacro">
     <xacro:macro name="flap">
+        <gazebo reference="flap_bottom">
+            <material>Gazebo/Green</material>
+        </gazebo>
+        <gazebo reference="flap_top">
+            <material>Gazebo/Green</material>
+        </gazebo>
+        <gazebo reference="board_expansion">
+            <material>Gazebo/DarkGrey</material>
+        </gazebo>
         <joint name="flap_bottom_joint" type="fixed">
             <origin xyz="-0.05 0 0" rpy="0 0 0" />
@@ -8,4 +17,9 @@
         </joint>
         <link name="flap_bottom">
+            <inertial>
+                <mass value="0.01"/>
+                <origin rpy=" 0 0 0" xyz="0 0 0"/>
+                <inertia ixx="1.6666666666666668e-07" ixy="0" ixz="0" iyy="1.6666666666666668e-07" iyz="0" izz="1.6666666666666668e-07"/>
+            </inertial>
             <visual>
                 <!--<origin xyz="-0.0161 0 0.009" rpy="0 0 0" />-->
@@ -20,4 +34,9 @@
         </joint>
         <link name="flap_top">
+            <inertial>
+                <mass value="0.01"/>
+                <origin rpy=" 0 0 0" xyz="0 0 0"/>
+                <inertia ixx="1.6666666666666668e-07" ixy="0" ixz="0" iyy="1.6666666666666668e-07" iyz="0" izz="1.6666666666666668e-07"/>
+            </inertial>
             <visual>
                 <!--<origin xyz="-0.0161 0 0.009" rpy="0 0 0" />-->
@@ -32,4 +51,9 @@
         </joint>
         <link name="board_expansion">
+            <inertial>
+                <mass value="0.01"/>
+                <origin rpy=" 0 0 0" xyz="0 0 0"/>
+                <inertia ixx="1.6666666666666668e-07" ixy="0" ixz="0" iyy="1.6666666666666668e-07" iyz="0" izz="1.6666666666666668e-07"/>
+            </inertial>
             <visual>
                 <!--<origin xyz="-0.0017 0 0.019" rpy="0 0 0" />-->

File: nanosaur_description/urdf/head/head_fisheye.urdf.xacro (robot description, xacro)
@@ -4,4 +4,16 @@
     <xacro:property name="display_angle" value="70.6"/>
     <xacro:macro name="nanosaur_head_fisheye">
+        <gazebo reference="cover">
+            <material>Gazebo/Green</material>
+        </gazebo>
+        <gazebo reference="display_left">
+            <material>Gazebo/Black</material>
+        </gazebo>
+        <gazebo reference="display_right">
+            <material>Gazebo/Black</material>
+        </gazebo>
+        <gazebo reference="camera_board">
+            <material>Gazebo/Grey</material>
+        </gazebo>
         <joint name="cover_joint" type="fixed">
             <origin xyz="0.06 0 -0.026" rpy="0 0 0" />
@@ -10,4 +22,9 @@
         </joint>
         <link name="cover">
+            <inertial>
+                <mass value="0.01"/>
+                <origin rpy=" 0 0 0" xyz="0 0 0"/>
+                <inertia ixx="1.6666666666666668e-07" ixy="0" ixz="0" iyy="1.6666666666666668e-07" iyz="0" izz="1.6666666666666668e-07"/>
+            </inertial>
             <visual>
                 <geometry><mesh filename="${path_meshes}/cover-fe.stl" scale="0.001 0.001 0.001"/></geometry>
@@ -21,4 +38,9 @@
         </joint>
         <link name="display_left">
+            <inertial>
+                <mass value="0.01"/>
+                <origin rpy=" 0 0 0" xyz="0 0 0"/>
+                <inertia ixx="1.6666666666666668e-07" ixy="0" ixz="0" iyy="1.6666666666666668e-07" iyz="0" izz="1.6666666666666668e-07"/>
+            </inertial>
             <visual>
                 <origin xyz="0 0 0" rpy="0 0 ${M_PI/2}" />
@@ -33,4 +55,9 @@
         </joint>
         <link name="display_right">
+            <inertial>
+                <mass value="0.01"/>
+                <origin rpy=" 0 0 0" xyz="0 0 0"/>
+                <inertia ixx="1.6666666666666668e-07" ixy="0" ixz="0" iyy="1.6666666666666668e-07" iyz="0" izz="1.6666666666666668e-07"/>
+            </inertial>
             <visual>
                 <origin xyz="0 0 0" rpy="0 0 ${M_PI/2}" />
@@ -45,4 +72,9 @@
         </joint>
         <link name="camera_board">
+            <inertial>
+                <mass value="0.01"/>
+                <origin rpy=" 0 0 0" xyz="0 0 0"/>
+                <inertia ixx="1.6666666666666668e-07" ixy="0" ixz="0" iyy="1.6666666666666668e-07" iyz="0" izz="1.6666666666666668e-07"/>
+            </inertial>
             <visual>
                 <origin xyz="-0.0039 0 -0.001" rpy="${M_PI/2} 0 -${M_PI/2}" />

File: nanosaur_description/urdf/head/head_pi.urdf.xacro (robot description, xacro)
@@ -4,4 +4,16 @@
     <xacro:property name="display_angle" value="70.6"/>
     <xacro:macro name="nanosaur_head_pi">
+        <gazebo reference="cover">
+            <material>Gazebo/Green</material>
+        </gazebo>
+        <gazebo reference="display_left">
+            <material>Gazebo/Black</material>
+        </gazebo>
+        <gazebo reference="display_right">
+            <material>Gazebo/Black</material>
+        </gazebo>
+        <gazebo reference="camera_board">
+            <material>Gazebo/Grey</material>
+        </gazebo>
         <joint name="cover_joint" type="fixed">
             <origin xyz="0.06 0 -0.026" rpy="0 0 0" />
@@ -10,4 +22,9 @@
         </joint>
         <link name="cover">
+            <inertial>
+                <mass value="0.01"/>
+                <origin rpy=" 0 0 0" xyz="0 0 0"/>
+                <inertia ixx="1.6666666666666668e-07" ixy="0" ixz="0" iyy="1.6666666666666668e-07" iyz="0" izz="1.6666666666666668e-07"/>
+            </inertial>
             <visual>
                 <geometry><mesh filename="${path_meshes}/cover.stl" scale="0.001 0.001 0.001"/></geometry>
@@ -21,4 +38,9 @@
         </joint>
         <link name="display_left">
+            <inertial>
+                <mass value="0.01"/>
+                <origin rpy=" 0 0 0" xyz="0 0 0"/>
+                <inertia ixx="1.6666666666666668e-07" ixy="0" ixz="0" iyy="1.6666666666666668e-07" iyz="0" izz="1.6666666666666668e-07"/>
+            </inertial>
             <visual>
                 <origin xyz="0 0 0" rpy="0 0 ${M_PI/2}" />
@@ -33,4 +55,9 @@
         </joint>
         <link name="display_right">
+            <inertial>
+                <mass value="0.01"/>
+                <origin rpy=" 0 0 0" xyz="0 0 0"/>
+                <inertia ixx="1.6666666666666668e-07" ixy="0" ixz="0" iyy="1.6666666666666668e-07" iyz="0" izz="1.6666666666666668e-07"/>
+            </inertial>
             <visual>
                 <origin xyz="0 0 0" rpy="0 0 ${M_PI/2}" />
@@ -45,4 +72,9 @@
         </joint>
         <link name="camera_board">
+            <inertial>
+                <mass value="0.01"/>
+                <origin rpy=" 0 0 0" xyz="0 0 0"/>
+                <inertia ixx="1.6666666666666668e-07" ixy="0" ixz="0" iyy="1.6666666666666668e-07" iyz="0" izz="1.6666666666666668e-07"/>
+            </inertial>
             <visual>
                 <origin xyz="-0.0025 0 0" rpy="0 0 ${M_PI}" />

File: nanosaur_description/urdf/head/head_realsense.urdf.xacro (robot description, xacro)
@@ -6,4 +6,13 @@
     <xacro:property name="display_angle" value="67"/>
     <xacro:macro name="nanosaur_head_realsense" params="name:=camera use_nominal_extrinsics:=false">
+        <gazebo reference="cover">
+            <material>Gazebo/Green</material>
+        </gazebo>
+        <gazebo reference="display_left">
+            <material>Gazebo/Black</material>
+        </gazebo>
+        <gazebo reference="display_right">
+            <material>Gazebo/Black</material>
+        </gazebo>
         <joint name="cover_joint" type="fixed">
             <origin xyz="0.06 0 -0.026" rpy="0 0 0" />
@@ -12,4 +21,9 @@
         </joint>
         <link name="cover">
+            <inertial>
+                <mass value="0.01"/>
+                <origin rpy=" 0 0 0" xyz="0 0 0"/>
+                <inertia ixx="1.6666666666666668e-07" ixy="0" ixz="0" iyy="1.6666666666666668e-07" iyz="0" izz="1.6666666666666668e-07"/>
+            </inertial>
             <visual>
                 <geometry><mesh filename="${path_meshes}/cover-rs.stl" scale="0.001 0.001 0.001"/></geometry>
@@ -23,4 +37,9 @@
         </joint>
         <link name="display_left">
+            <inertial>
+                <mass value="0.01"/>
+                <origin rpy=" 0 0 0" xyz="0 0 0"/>
+                <inertia ixx="1.6666666666666668e-07" ixy="0" ixz="0" iyy="1.6666666666666668e-07" iyz="0" izz="1.6666666666666668e-07"/>
+            </inertial>
             <visual>
                 <origin xyz="0 0 0" rpy="0 0 ${M_PI/2}" />
@@ -35,4 +54,9 @@
         </joint>
         <link name="display_right">
+            <inertial>
+                <mass value="0.01"/>
+                <origin rpy=" 0 0 0" xyz="0 0 0"/>
+                <inertia ixx="1.6666666666666668e-07" ixy="0" ixz="0" iyy="1.6666666666666668e-07" iyz="0" izz="1.6666666666666668e-07"/>
+            </inertial>
             <visual>
                 <origin xyz="0 0 0" rpy="0 0 ${M_PI/2}" />

File: nanosaur_description/urdf/head/head_zedmini.urdf.xacro (robot description, xacro)
@@ -5,4 +5,13 @@
     <xacro:property name="display_angle" value="67"/>
     <xacro:macro name="nanosaur_head_zedmini" params="name:=zed">
+        <gazebo reference="cover">
+            <material>Gazebo/Green</material>
+        </gazebo>
+        <gazebo reference="display_left">
+            <material>Gazebo/Black</material>
+        </gazebo>
+        <gazebo reference="display_right">
+            <material>Gazebo/Black</material>
+        </gazebo>
         <joint name="cover_joint" type="fixed">
             <origin xyz="0.06 0 -0.026" rpy="0 0 0" />
@@ -11,4 +20,9 @@
         </joint>
         <link name="cover">
+            <inertial>
+                <mass value="0.01"/>
+                <origin rpy=" 0 0 0" xyz="0 0 0"/>
+                <inertia ixx="1.6666666666666668e-07" ixy="0" ixz="0" iyy="1.6666666666666668e-07" iyz="0" izz="1.6666666666666668e-07"/>
+            </inertial>
             <visual>
                 <geometry><mesh filename="${path_meshes}/cover-zedmini.stl" scale="0.001 0.001 0.001"/></geometry>
@@ -22,4 +36,9 @@
         </joint>
         <link name="display_left">
+            <inertial>
+                <mass value="0.01"/>
+                <origin rpy=" 0 0 0" xyz="0 0 0"/>
+                <inertia ixx="1.6666666666666668e-07" ixy="0" ixz="0" iyy="1.6666666666666668e-07" iyz="0" izz="1.6666666666666668e-07"/>
+            </inertial>
             <visual>
                 <origin xyz="0 0 0" rpy="0 0 ${M_PI/2}" />
@@ -34,4 +53,9 @@
         </joint>
         <link name="display_right">
+            <inertial>
+                <mass value="0.01"/>
+                <origin rpy=" 0 0 0" xyz="0 0 0"/>
+                <inertia ixx="1.6666666666666668e-07" ixy="0" ixz="0" iyy="1.6666666666666668e-07" iyz="0" izz="1.6666666666666668e-07"/>
+            </inertial>
             <visual>
                 <origin xyz="0 0 0" rpy="0 0 ${M_PI/2}" />

File: nanosaur_description/urdf/head/zedmini.urdf.xacro (robot description, xacro)
@@ -2,4 +2,7 @@
 <robot xmlns:xacro="http://wiki.ros.org/xacro">
   <xacro:macro name="zed_camera" params="name=zed model=zedm parent *origin">
+    <gazebo reference="${name}_camera_center">
+        <material>Gazebo/Black</material>
+    </gazebo>
     <xacro:if value="${model == 'zedm'}">
       <xacro:property name="baseline" value="0.06" />

File: nanosaur_description/urdf/track.urdf.xacro (robot description, xacro)
@@ -1,5 +1,28 @@
 <?xml version="1.0"?>
 <robot name="nanosaur_track" xmlns:xacro="http://ros.org/wiki/xacro">
-    <xacro:macro name="track" params="type parent radius">
+    <xacro:macro name="track" params="type parent radius simulation">
+        <gazebo reference="sprocket_${type}">
+            <kp>10000000</kp>
+            <kd>10000000</kd>
+            <mu1>10000000</mu1>
+            <mu2>10000000</mu2>
+            <material>Gazebo/Blue</material>
+        </gazebo>
+        <gazebo reference="motor_${type}">
+            <material>Gazebo/Gold</material>
+        </gazebo>
+        <gazebo reference="wheel_${type}">
+            <kp>10000000</kp>
+            <kd>10000000</kd>
+            <mu1>0</mu1>
+            <mu2>0</mu2>
+            <material>Gazebo/Red</material>
+        </gazebo>
+        <gazebo reference="track_${type}">
+            <material>Gazebo/Black</material>
+        </gazebo>
+        <gazebo reference="slider_${type}">
+            <material>Gazebo/Green</material>
+        </gazebo>
         <!-- Define orientation -->
         <xacro:if value="${type == 'left'}">
@@ -10,5 +33,10 @@
         </xacro:if>
         <joint name="sprocket_${type}_joint" type="continuous">
-            <origin xyz="0.053 ${orientation * -0.043} 0.015" rpy="${orientation * M_PI/2} 0 0" />
+            <xacro:if value="${simulation}">
+                <origin xyz="0.0 ${orientation * -0.043} 0.015" rpy="${orientation * M_PI/2} 0 0" />
+            </xacro:if>
+            <xacro:unless value="${simulation}">
+                <origin xyz="0.053 ${orientation * -0.043} 0.015" rpy="${orientation * M_PI/2} 0 0" />
+            </xacro:unless>
             <parent link="${parent}"/>
             <child link="sprocket_${type}"/>
@@ -16,4 +44,9 @@
         </joint>
         <link name="sprocket_${type}">
+            <inertial>
+                <mass value="0.01"/>
+                <origin rpy=" 0 0 0" xyz="0 0 0"/>
+                <inertia ixx="1.6666666666666668e-07" ixy="0" ixz="0" iyy="1.6666666666666668e-07" iyz="0" izz="1.6666666666666668e-07"/>
+            </inertial>
             <visual>
                 <origin xyz="0 0 0" rpy="0 0 0" />
@@ -49,4 +82,9 @@
         </joint>
         <link name="wheel_${type}">
+            <inertial>
+                <mass value="0.01"/>
+                <origin rpy=" 0 0 0" xyz="0 0 0"/>
+                <inertia ixx="1.6666666666666668e-07" ixy="0" ixz="0" iyy="1.6666666666666668e-07" iyz="0" izz="1.6666666666666668e-07"/>
+            </inertial>
             <visual>
                 <origin xyz="0 0 0" rpy="0 0 0" />
@@ -61,4 +99,38 @@
             </collision>
         </link>
+        <xacro:if value="${simulation}">
+            <joint name="front_wheel_${type}_joint" type="fixed">
+                <origin xyz="0 0 0" rpy="0 0 0" />
+                <parent link="motor_${type}"/>
+                <child link="front_wheel_${type}"/>
+                <!-- Passive sprocket rotate automatically according to the status of the active one -->
+                <mimic joint="sprocket_${type}_joint" multiplier="1" offset="0"/>
+            </joint>
+            <link name="front_wheel_${type}">
+                <inertial>
+                    <mass value="0.01"/>
+                    <origin rpy=" 0 0 0" xyz="0 0 0"/>
+                    <inertia ixx="1.6666666666666668e-07" ixy="0" ixz="0" iyy="1.6666666666666668e-07" iyz="0" izz="1.6666666666666668e-07"/>
+                </inertial>
+                <visual>
+                    <origin xyz="0 0 0" rpy="0 0 0" />
+                    <geometry><mesh filename="${path_meshes}/wheel.stl" scale="0.001 0.001 0.001"/></geometry>
+                    <material name="Black" />
+                </visual>
+                <!-- Collision cylinder -->
+                <collision>
+                    <origin xyz="0 0 0" rpy="0 0 0" />
+                    <geometry><cylinder length="0.015" radius="${radius}"/></geometry>
+                    <material name="Black" />
+                </collision>
+            </link>
+            <gazebo reference="front_wheel_${type}">
+                <kp>10000000</kp>
+                <kd>10000000</kd>
+                <mu1>0</mu1>
+                <mu2>0</mu2>
+                <material>Gazebo/Green</material>
+            </gazebo>
+        </xacro:if>
         <joint name="track_${type}_joint" type="fixed">
             <origin xyz="-0.049 0 0" rpy="0 0 0" />
@@ -67,4 +139,9 @@
         </joint>
         <link name="track_${type}">
+            <inertial>
+                <mass value="0.01"/>
+                <origin rpy=" 0 0 0" xyz="0 0 0"/>
+                <inertia ixx="1.6666666666666668e-07" ixy="0" ixz="0" iyy="1.6666666666666668e-07" iyz="0" izz="1.6666666666666668e-07"/>
+            </inertial>
             <visual>
                 <origin xyz="0 0 0" rpy="${M_PI/2} 0 0" />
@@ -78,4 +155,9 @@
         </joint>
         <link name="slider_${type}">
+            <inertial>
+                <mass value="0.01"/>
+                <origin rpy=" 0 0 0" xyz="0 0 0"/>
+                <inertia ixx="1.6666666666666668e-07" ixy="0" ixz="0" iyy="1.6666666666666668e-07" iyz="0" izz="1.6666666666666668e-07"/>
+            </inertial>
             <visual>
                 <origin xyz="0 0 0.008" rpy="0 0 0" />
