Commit message: Fix xacro for Ignition

File: nanosaur_description/urdf/flap.urdf.xacro (robot description, xacro)
@@ -1,13 +1,38 @@
 <?xml version="1.0"?>
-<robot name="nanosaur_flap" xmlns:xacro="http://ros.org/wiki/xacro">
+<robot name="nanosaur_flap"
+    xmlns:xacro="http://ros.org/wiki/xacro">
     <xacro:macro name="flap">
         <gazebo reference="flap_bottom">
             <material>Gazebo/Green</material>
+            <!-- Ignition color reference -->
+            <visual>
+                <material>
+                    <ambient>0.0 0.5 0.0 1.0</ambient>
+                    <diffuse>0.0 0.5 0.0 1.0</diffuse>
+                    <specular>0.0 0.5 0.0 1.0</specular>
+                </material>
+            </visual>
         </gazebo>
         <gazebo reference="flap_top">
             <material>Gazebo/Green</material>
+            <!-- Ignition color reference -->
+            <visual>
+                <material>
+                    <ambient>0.0 0.5 0.0 1.0</ambient>
+                    <diffuse>0.0 0.5 0.0 1.0</diffuse>
+                    <specular>0.0 0.5 0.0 1.0</specular>
+                </material>
+            </visual>
         </gazebo>
         <gazebo reference="board_expansion">
             <material>Gazebo/DarkGrey</material>
+            <!-- Ignition color reference -->
+            <visual>
+                <material>
+                    <ambient>0.5 0.5 0.5 1.0</ambient>
+                    <diffuse>0.5 0.5 0.5 1.0</diffuse>
+                    <specular>0.5 0.5 0.5 1.0</specular>
+                </material>
+            </visual>
         </gazebo>
         <joint name="flap_bottom_joint" type="fixed">
@@ -25,5 +50,7 @@
                 <!--<origin xyz="-0.0161 0 0.009" rpy="0 0 0" />-->
                 <origin xyz="0.0068 0 0.0175" rpy="0 0 0" />
-                <geometry><mesh filename="${path_meshes}/flap_bottom.stl" scale="0.001 0.001 0.001"/></geometry>
+                <geometry>
+                    <mesh filename="${path_meshes}/flap_bottom.stl" scale="0.001 0.001 0.001"/>
+                </geometry>
                 <material name="Green" />
             </visual>
@@ -42,5 +69,7 @@
                 <!--<origin xyz="-0.0161 0 0.009" rpy="0 0 0" />-->
                 <origin xyz="0.0068 0 0.0175" rpy="0 0 0" />
-                <geometry><mesh filename="${path_meshes}/flap_top.stl" scale="0.001 0.001 0.001"/></geometry>
+                <geometry>
+                    <mesh filename="${path_meshes}/flap_top.stl" scale="0.001 0.001 0.001"/>
+                </geometry>
                 <material name="Green" />
             </visual>
@@ -59,5 +88,7 @@
                 <!--<origin xyz="-0.0017 0 0.019" rpy="0 0 0" />-->
                 <origin xyz="-0.002 0.0005 0.017" rpy="0 0 0" />
-                <geometry><mesh filename="${path_meshes}/parts/nanosaur-exp-board.stl"/></geometry>
+                <geometry>
+                    <mesh filename="${path_meshes}/parts/nanosaur-exp-board.stl"/>
+                </geometry>
                 <material name="GunMetalGrey" />
             </visual>

File: nanosaur_description/urdf/head/head_fisheye.urdf.xacro (robot description, xacro)
@@ -1,4 +1,5 @@
 <?xml version="1.0"?>
-<robot name="nanosaur_head_fisheye" xmlns:xacro="http://ros.org/wiki/xacro">
+<robot name="nanosaur_head_fisheye"
+    xmlns:xacro="http://ros.org/wiki/xacro">
     <xacro:property name="cam_angle" value="5"/>
     <xacro:property name="display_angle" value="70.6"/>
@@ -6,4 +7,12 @@
         <gazebo reference="cover">
             <material>Gazebo/Green</material>
+            <!-- Ignition color reference -->
+            <visual>
+                <material>
+                    <ambient>0.0 0.5 0.0 1.0</ambient>
+                    <diffuse>0.0 0.5 0.0 1.0</diffuse>
+                    <specular>0.0 0.5 0.0 1.0</specular>
+                </material>
+            </visual>
         </gazebo>
         <gazebo reference="display_left">
@@ -15,4 +24,12 @@
         <gazebo reference="camera_board">
             <material>Gazebo/Grey</material>
+            <!-- Ignition color reference -->
+            <visual>
+                <material>
+                    <ambient>0.2 0.2 0.2 1.0</ambient>
+                    <diffuse>0.2 0.2 0.2 1.0</diffuse>
+                    <specular>0.2 0.2 0.2 1.0</specular>
+                </material>
+            </visual>
         </gazebo>
         <joint name="cover_joint" type="fixed">
@@ -28,5 +45,7 @@
             </inertial>
             <visual>
-                <geometry><mesh filename="${path_meshes}/cover-fe.stl" scale="0.001 0.001 0.001"/></geometry>
+                <geometry>
+                    <mesh filename="${path_meshes}/cover-fe.stl" scale="0.001 0.001 0.001"/>
+                </geometry>
                 <material name="Green" />
             </visual>
@@ -34,5 +53,7 @@
             <collision>
                 <origin xyz="0.003 0 0.03" rpy="${M_PI/2} ${M_PI/2} 0" />
-                <geometry><cylinder length="0.07" radius="0.028"/></geometry>
+                <geometry>
+                    <cylinder length="0.07" radius="0.028"/>
+                </geometry>
                 <material name="Green" />
             </collision>
@@ -51,5 +72,7 @@
             <visual>
                 <origin xyz="0 0 0" rpy="0 0 ${M_PI/2}" />
-                <geometry><mesh filename="${path_meshes}/parts/OLED_Module.stl"/></geometry>
+                <geometry>
+                    <mesh filename="${path_meshes}/parts/OLED_Module.stl"/>
+                </geometry>
                 <material name="Black" />
             </visual>
@@ -68,5 +91,7 @@
             <visual>
                 <origin xyz="0 0 0" rpy="0 0 ${M_PI/2}" />
-                <geometry><mesh filename="${path_meshes}/parts/OLED_Module.stl"/></geometry>
+                <geometry>
+                    <mesh filename="${path_meshes}/parts/OLED_Module.stl"/>
+                </geometry>
                 <material name="Black" />
             </visual>
@@ -85,5 +110,7 @@
             <visual>
                 <origin xyz="-0.0039 0 -0.001" rpy="${M_PI/2} 0 -${M_PI/2}" />
-                <geometry><mesh filename="${path_meshes}/parts/fisheye_camera.dae"/></geometry>
+                <geometry>
+                    <mesh filename="${path_meshes}/parts/fisheye_camera.dae"/>
+                </geometry>
             </visual>
         </link>

File: nanosaur_description/urdf/head/head_pi.urdf.xacro (robot description, xacro)
@@ -1,4 +1,5 @@
 <?xml version="1.0"?>
-<robot name="nanosaur_head_pi" xmlns:xacro="http://ros.org/wiki/xacro">
+<robot name="nanosaur_head_pi"
+    xmlns:xacro="http://ros.org/wiki/xacro">
     <xacro:property name="cam_angle" value="5"/>
     <xacro:property name="display_angle" value="70.6"/>
@@ -6,4 +7,12 @@
         <gazebo reference="cover">
             <material>Gazebo/Green</material>
+            <!-- Ignition color reference -->
+            <visual>
+                <material>
+                    <ambient>0.0 0.5 0.0 1.0</ambient>
+                    <diffuse>0.0 0.5 0.0 1.0</diffuse>
+                    <specular>0.0 0.5 0.0 1.0</specular>
+                </material>
+            </visual>
         </gazebo>
         <gazebo reference="display_left">
@@ -15,4 +24,12 @@
         <gazebo reference="camera_board">
             <material>Gazebo/Grey</material>
+            <!-- Ignition color reference -->
+            <visual>
+                <material>
+                    <ambient>0.2 0.2 0.2 1.0</ambient>
+                    <diffuse>0.2 0.2 0.2 1.0</diffuse>
+                    <specular>0.2 0.2 0.2 1.0</specular>
+                </material>
+            </visual>
         </gazebo>
         <joint name="cover_joint" type="fixed">
@@ -28,5 +45,7 @@
             </inertial>
             <visual>
-                <geometry><mesh filename="${path_meshes}/cover.stl" scale="0.001 0.001 0.001"/></geometry>
+                <geometry>
+                    <mesh filename="${path_meshes}/cover.stl" scale="0.001 0.001 0.001"/>
+                </geometry>
                 <material name="Green" />
             </visual>
@@ -34,5 +53,7 @@
             <collision>
                 <origin xyz="-0.007 0 0.03" rpy="${M_PI/2} ${M_PI/2} 0" />
-                <geometry><cylinder length="0.07" radius="0.028"/></geometry>
+                <geometry>
+                    <cylinder length="0.07" radius="0.028"/>
+                </geometry>
                 <material name="Green" />
             </collision>
@@ -51,5 +72,7 @@
             <visual>
                 <origin xyz="0 0 0" rpy="0 0 ${M_PI/2}" />
-                <geometry><mesh filename="${path_meshes}/parts/OLED_Module.stl"/></geometry>
+                <geometry>
+                    <mesh filename="${path_meshes}/parts/OLED_Module.stl"/>
+                </geometry>
                 <material name="Black" />
             </visual>
@@ -68,5 +91,7 @@
             <visual>
                 <origin xyz="0 0 0" rpy="0 0 ${M_PI/2}" />
-                <geometry><mesh filename="${path_meshes}/parts/OLED_Module.stl"/></geometry>
+                <geometry>
+                    <mesh filename="${path_meshes}/parts/OLED_Module.stl"/>
+                </geometry>
                 <material name="Black" />
             </visual>
@@ -85,5 +110,7 @@
             <visual>
                 <origin xyz="-0.0025 0 0" rpy="0 0 ${M_PI}" />
-                <geometry><mesh filename="${path_meshes}/parts/rasp_camera.stl"/></geometry>
+                <geometry>
+                    <mesh filename="${path_meshes}/parts/rasp_camera.stl"/>
+                </geometry>
                 <material name="aluminum" />
             </visual>

File: nanosaur_description/urdf/head/head_realsense.urdf.xacro (robot description, xacro)
@@ -1,4 +1,5 @@
 <?xml version="1.0"?>
-<robot name="nanosaur_head_realsense" xmlns:xacro="http://ros.org/wiki/xacro">
+<robot name="nanosaur_head_realsense"
+    xmlns:xacro="http://ros.org/wiki/xacro">
     <xacro:include filename="$(find nanosaur_description)/urdf/head/d435.urdf.xacro" />
     <xacro:include filename="$(find nanosaur_description)/urdf/head/d435i_imu_modules.urdf.xacro"/>
@@ -8,4 +9,12 @@
         <gazebo reference="cover">
             <material>Gazebo/Green</material>
+            <!-- Ignition color reference -->
+            <visual>
+                <material>
+                    <ambient>0.0 0.5 0.0 1.0</ambient>
+                    <diffuse>0.0 0.5 0.0 1.0</diffuse>
+                    <specular>0.0 0.5 0.0 1.0</specular>
+                </material>
+            </visual>
         </gazebo>
         <gazebo reference="display_left">
@@ -27,5 +36,7 @@
             </inertial>
             <visual>
-                <geometry><mesh filename="${path_meshes}/cover-rs.stl" scale="0.001 0.001 0.001"/></geometry>
+                <geometry>
+                    <mesh filename="${path_meshes}/cover-rs.stl" scale="0.001 0.001 0.001"/>
+                </geometry>
                 <material name="Green" />
             </visual>
@@ -33,5 +44,7 @@
             <collision>
                 <origin xyz="0.003 0 0.03" rpy="${M_PI/2} ${M_PI/2} 0" />
-                <geometry><cylinder length="0.07" radius="0.028"/></geometry>
+                <geometry>
+                    <cylinder length="0.07" radius="0.028"/>
+                </geometry>
                 <material name="Green" />
             </collision>
@@ -50,5 +63,7 @@
             <visual>
                 <origin xyz="0 0 0" rpy="0 0 ${M_PI/2}" />
-                <geometry><mesh filename="${path_meshes}/parts/OLED_Module.stl"/></geometry>
+                <geometry>
+                    <mesh filename="${path_meshes}/parts/OLED_Module.stl"/>
+                </geometry>
                 <material name="Black" />
             </visual>
@@ -67,5 +82,7 @@
             <visual>
                 <origin xyz="0 0 0" rpy="0 0 ${M_PI/2}" />
-                <geometry><mesh filename="${path_meshes}/parts/OLED_Module.stl"/></geometry>
+                <geometry>
+                    <mesh filename="${path_meshes}/parts/OLED_Module.stl"/>
+                </geometry>
                 <material name="Black" />
             </visual>

File: nanosaur_description/urdf/head/head_zedmini.urdf.xacro (robot description, xacro)
@@ -1,4 +1,5 @@
 <?xml version="1.0"?>
-<robot name="nanosaur_head_zedmini" xmlns:xacro="http://ros.org/wiki/xacro">
+<robot name="nanosaur_head_zedmini"
+    xmlns:xacro="http://ros.org/wiki/xacro">
     <xacro:include filename="$(find nanosaur_description)/urdf/head/zedmini.urdf.xacro" />
     <xacro:property name="cam_angle" value="5"/>
@@ -7,4 +8,12 @@
         <gazebo reference="cover">
             <material>Gazebo/Green</material>
+            <!-- Ignition color reference -->
+            <visual>
+                <material>
+                    <ambient>0.0 0.5 0.0 1.0</ambient>
+                    <diffuse>0.0 0.5 0.0 1.0</diffuse>
+                    <specular>0.0 0.5 0.0 1.0</specular>
+                </material>
+            </visual>
         </gazebo>
         <gazebo reference="display_left">
@@ -26,5 +35,7 @@
             </inertial>
             <visual>
-                <geometry><mesh filename="${path_meshes}/cover-zedmini.stl" scale="0.001 0.001 0.001"/></geometry>
+                <geometry>
+                    <mesh filename="${path_meshes}/cover-zedmini.stl" scale="0.001 0.001 0.001"/>
+                </geometry>
                 <material name="Green" />
             </visual>
@@ -32,5 +43,7 @@
             <collision>
                 <origin xyz="0.003 0 0.03" rpy="${M_PI/2} ${M_PI/2} 0" />
-                <geometry><cylinder length="0.07" radius="0.028"/></geometry>
+                <geometry>
+                    <cylinder length="0.07" radius="0.028"/>
+                </geometry>
                 <material name="Green" />
             </collision>
@@ -49,5 +62,7 @@
             <visual>
                 <origin xyz="0 0 0" rpy="0 0 ${M_PI/2}" />
-                <geometry><mesh filename="${path_meshes}/parts/OLED_Module.stl"/></geometry>
+                <geometry>
+                    <mesh filename="${path_meshes}/parts/OLED_Module.stl"/>
+                </geometry>
                 <material name="Black" />
             </visual>
@@ -66,5 +81,7 @@
             <visual>
                 <origin xyz="0 0 0" rpy="0 0 ${M_PI/2}" />
-                <geometry><mesh filename="${path_meshes}/parts/OLED_Module.stl"/></geometry>
+                <geometry>
+                    <mesh filename="${path_meshes}/parts/OLED_Module.stl"/>
+                </geometry>
                 <material name="Black" />
             </visual>

File: nanosaur_description/urdf/robot.urdf.xacro (robot description, xacro)
@@ -22,24 +22,7 @@
         <!-- Gazebo color reference
         https://bitbucket.org/osrf/gazebo/src/default/media/materials/scripts/gazebo.material?fileviewer=file-view-default
-        http://wiki.ros.org/simulator_gazebo/Tutorials/ListOfMaterials
+        Gazebo http://wiki.ros.org/simulator_gazebo/Tutorials/ListOfMaterials
+        Ignition https://gazebosim.org/api/gazebo/3.7/migrationsdf.html
         -->
-        <gazebo reference="base_front">
-            <material>Gazebo/Green</material>
-        </gazebo>
-        <gazebo reference="base_rear">
-            <material>Gazebo/Green</material>
-        </gazebo>
-        <gazebo reference="motor_board">
-            <material>Gazebo/DarkGrey</material>
-        </gazebo>
-        <gazebo reference="power_bank">
-            <material>Gazebo/DarkGrey</material>
-        </gazebo>
-        <gazebo reference="pb_holder">
-            <material>Gazebo/Green</material>
-        </gazebo>
-        <gazebo reference="NVIDIA_jetson">
-            <material>Gazebo/DarkGrey</material>
-        </gazebo>
         <!-- nanosaur definition -->
         <link name="base_link" />

File: nanosaur_description/urdf/track.urdf.xacro (robot description, xacro)
@@ -1,4 +1,5 @@
 <?xml version="1.0"?>
-<robot name="nanosaur_track" xmlns:xacro="http://ros.org/wiki/xacro">
+<robot name="nanosaur_track"
+    xmlns:xacro="http://ros.org/wiki/xacro">
     <xacro:macro name="track" params="type parent radius diff_drive_emulation">
         <!-- Define orientation -->
@@ -28,5 +29,7 @@
             <visual>
                 <origin xyz="0 0 0" rpy="0 0 0" />
-                <geometry><mesh filename="${path_meshes}/sprocket.stl" scale="0.001 0.001 0.001"/></geometry>
+                <geometry>
+                    <mesh filename="${path_meshes}/sprocket.stl" scale="0.001 0.001 0.001"/>
+                </geometry>
                 <material name="Black" />
             </visual>
@@ -34,5 +37,7 @@
             <collision>
                 <origin xyz="0 0 0" rpy="0 0 0" />
-                <geometry><cylinder length="0.015" radius="${radius}"/></geometry>
+                <geometry>
+                    <cylinder length="0.015" radius="${radius}"/>
+                </geometry>
                 <material name="Black" />
             </collision>
@@ -44,4 +49,12 @@
             <mu2>10000000</mu2>
             <material>Gazebo/Blue</material>
+            <!-- Ignition color reference -->
+            <visual>
+                <material>
+                    <ambient>0.0 0.0 0.5 1.0</ambient>
+                    <diffuse>0.0 0.0 0.5 1.0</diffuse>
+                    <specular>0.0 0.0 0.5 1.0</specular>
+                </material>
+            </visual>
         </gazebo>
         <joint name="motor_${type}_joint" type="fixed">
@@ -53,5 +66,7 @@
             <visual>
                 <origin xyz="0 0 -0.031" rpy="0 0 -${M_PI/2}" />
-                <geometry><mesh filename="${path_meshes}/parts/Pololu-Micro-Metal-Gearmotor.stl"/></geometry>
+                <geometry>
+                    <mesh filename="${path_meshes}/parts/Pololu-Micro-Metal-Gearmotor.stl"/>
+                </geometry>
                 <material name="Gold" />
             </visual>
@@ -59,4 +74,12 @@
         <gazebo reference="motor_${type}">
             <material>Gazebo/Gold</material>
+            <!-- Ignition color reference -->
+            <visual>
+                <material>
+                    <ambient>0.9 0.7 0.0 1.0</ambient>
+                    <diffuse>0.9 0.7 0.0 1.0</diffuse>
+                    <specular>0.9 0.7 0.0 1.0</specular>
+                </material>
+            </visual>
         </gazebo>
         <joint name="wheel_${type}_joint" type="continuous">
@@ -76,5 +99,7 @@
             <visual>
                 <origin xyz="0 0 0" rpy="0 0 0" />
-                <geometry><mesh filename="${path_meshes}/wheel.stl" scale="0.001 0.001 0.001"/></geometry>
+                <geometry>
+                    <mesh filename="${path_meshes}/wheel.stl" scale="0.001 0.001 0.001"/>
+                </geometry>
                 <material name="Black" />
             </visual>
@@ -82,5 +107,7 @@
             <collision>
                 <origin xyz="0 0 0" rpy="0 0 0" />
-                <geometry><cylinder length="0.015" radius="${radius}"/></geometry>
+                <geometry>
+                    <cylinder length="0.015" radius="${radius}"/>
+                </geometry>
                 <material name="Black" />
             </collision>
@@ -92,4 +119,12 @@
             <mu2>0</mu2>
             <material>Gazebo/Red</material>
+            <!-- Ignition color reference -->
+            <visual>
+                <material>
+                    <ambient>0.5 0.0 0.0 1.0</ambient>
+                    <diffuse>0.5 0.0 0.0 1.0</diffuse>
+                    <specular>0.5 0.0 0.0 1.0</specular>
+                </material>
+            </visual>
         </gazebo>
         <xacro:if value="${diff_drive_emulation}">
@@ -109,5 +144,7 @@
                 <visual>
                     <origin xyz="0 0 0" rpy="0 0 0" />
-                    <geometry><mesh filename="${path_meshes}/wheel.stl" scale="0.001 0.001 0.001"/></geometry>
+                    <geometry>
+                        <mesh filename="${path_meshes}/wheel.stl" scale="0.001 0.001 0.001"/>
+                    </geometry>
                     <material name="Black" />
                 </visual>
@@ -115,5 +152,7 @@
                 <collision>
                     <origin xyz="0 0 0" rpy="0 0 0" />
-                    <geometry><cylinder length="0.015" radius="${radius}"/></geometry>
+                    <geometry>
+                        <cylinder length="0.015" radius="${radius}"/>
+                    </geometry>
                     <material name="Black" />
                 </collision>
@@ -125,4 +164,12 @@
                 <mu2>0</mu2>
                 <material>Gazebo/Green</material>
+                <!-- Ignition color reference -->
+                <visual>
+                    <material>
+                        <ambient>0.0 0.5 0.0 1.0</ambient>
+                        <diffuse>0.0 0.5 0.0 1.0</diffuse>
+                        <specular>0.0 0.5 0.0 1.0</specular>
+                    </material>
+                </visual>
             </gazebo>
         </xacro:if>
@@ -140,5 +187,7 @@
             <visual>
                 <origin xyz="0 0 0" rpy="${M_PI/2} 0 0" />
-                <geometry><mesh filename="${path_meshes}/track.stl" scale="0.001 0.001 0.001"/></geometry>
+                <geometry>
+                    <mesh filename="${path_meshes}/track.stl" scale="0.001 0.001 0.001"/>
+                </geometry>
                 <material name="Black" />
             </visual>
@@ -146,4 +195,12 @@
         <gazebo reference="track_${type}">
             <material>Gazebo/Black</material>
+            <!-- Ignition color reference -->
+            <visual>
+                <material>
+                    <ambient>0.01 0.01 0.01 1.0</ambient>
+                    <diffuse>0.01 0.01 0.01 1.0</diffuse>
+                    <specular>0.01 0.01 0.01 1.0</specular>
+                </material>
+            </visual>
         </gazebo>
         <joint name="slider_${type}_joint" type="fixed">
@@ -159,5 +216,7 @@
             <visual>
                 <origin xyz="0 0 0.008" rpy="0 0 0" />
-                <geometry><mesh filename="${path_meshes}/slider.stl" scale="0.001 0.001 0.001"/></geometry>
+                <geometry>
+                    <mesh filename="${path_meshes}/slider.stl" scale="0.001 0.001 0.001"/>
+                </geometry>
                 <material name="Green" />
             </visual>
@@ -165,4 +224,12 @@
         <gazebo reference="slider_${type}">
             <material>Gazebo/Green</material>
+            <!-- Ignition color reference -->
+            <visual>
+                <material>
+                    <ambient>0.0 0.5 0.0 1.0</ambient>
+                    <diffuse>0.0 0.5 0.0 1.0</diffuse>
+                    <specular>0.0 0.5 0.0 1.0</specular>
+                </material>
+            </visual>
         </gazebo>
     </xacro:macro>
