Commit message: rename variable simulation to diff_drive_emulation

File: nanosaur_description/urdf/robot.urdf.xacro (robot description, xacro)
@@ -16,35 +16,29 @@
     <!-- nanosaur properties -->
     <xacro:property name="motor_board_angle" value="35"/>
-    <xacro:macro name="nanosaur" params="cover_type use_nominal_extrinsics simulation">
-        <xacro:if value="${simulation}">
-            <!-- Gazebo color reference
-            https://bitbucket.org/osrf/gazebo/src/default/media/materials/scripts/gazebo.material?fileviewer=file-view-default
-            http://wiki.ros.org/simulator_gazebo/Tutorials/ListOfMaterials
-            -->
-            <gazebo reference="base_front">
-                <material>Gazebo/Green</material>
-            </gazebo>
-            <gazebo reference="base_rear">
-                <material>Gazebo/Green</material>
-            </gazebo>
-            <gazebo reference="motor_board">
-                <material>Gazebo/DarkGrey</material>
-            </gazebo>
-            <gazebo reference="power_bank">
-                <material>Gazebo/DarkGrey</material>
-            </gazebo>
-            <gazebo reference="pb_holder">
-                <material>Gazebo/Green</material>
-            </gazebo>
-            <gazebo reference="NVIDIA_jetson">
-                <material>Gazebo/DarkGrey</material>
-            </gazebo>
-            <!-- nanosaur properties -->
-            <xacro:property name="sprocket_radius" value="0.0150"/>
-        </xacro:if>
-        <xacro:unless value="${simulation}">
-            <!-- nanosaur properties -->
-            <xacro:property name="sprocket_radius" value="0.0105"/>
-        </xacro:unless>
+    <!-- Real radius 0.0105 but augmented for track thickness -->
+    <xacro:property name="sprocket_radius" value="0.0150"/>
+    <xacro:macro name="nanosaur" params="cover_type use_nominal_extrinsics diff_drive_emulation">
+        <!-- Gazebo color reference
+        https://bitbucket.org/osrf/gazebo/src/default/media/materials/scripts/gazebo.material?fileviewer=file-view-default
+        http://wiki.ros.org/simulator_gazebo/Tutorials/ListOfMaterials
+        -->
+        <gazebo reference="base_front">
+            <material>Gazebo/Green</material>
+        </gazebo>
+        <gazebo reference="base_rear">
+            <material>Gazebo/Green</material>
+        </gazebo>
+        <gazebo reference="motor_board">
+            <material>Gazebo/DarkGrey</material>
+        </gazebo>
+        <gazebo reference="power_bank">
+            <material>Gazebo/DarkGrey</material>
+        </gazebo>
+        <gazebo reference="pb_holder">
+            <material>Gazebo/Green</material>
+        </gazebo>
+        <gazebo reference="NVIDIA_jetson">
+            <material>Gazebo/DarkGrey</material>
+        </gazebo>
         <!-- nanosaur definition -->
         <link name="base_link" />
@@ -153,6 +147,6 @@
             </visual>
         </link>
-        <xacro:track type="left" parent="base_link" radius="${sprocket_radius}" simulation="${simulation}"/>
-        <xacro:track type="right" parent="base_link" radius="${sprocket_radius}" simulation="${simulation}"/>
+        <xacro:track type="left" parent="base_link" radius="${sprocket_radius}" diff_drive_emulation="${diff_drive_emulation}"/>
+        <xacro:track type="right" parent="base_link" radius="${sprocket_radius}" diff_drive_emulation="${diff_drive_emulation}"/>
         <xacro:flap />
         <!-- Nanosaur heads -->

File: nanosaur_description/urdf/track.urdf.xacro (robot description, xacro)
@@ -1,5 +1,5 @@
 <?xml version="1.0"?>
 <robot name="nanosaur_track" xmlns:xacro="http://ros.org/wiki/xacro">
-    <xacro:macro name="track" params="type parent radius simulation">
+    <xacro:macro name="track" params="type parent radius diff_drive_emulation">
         <!-- Define orientation -->
         <xacro:if value="${type == 'left'}">
@@ -10,8 +10,8 @@
         </xacro:if>
         <joint name="sprocket_${type}_joint" type="continuous">
-            <xacro:if value="${simulation}">
+            <xacro:if value="${diff_drive_emulation}">
                 <origin xyz="0.0 ${orientation * -0.043} 0.015" rpy="${orientation * M_PI/2} 0 0" />
             </xacro:if>
-            <xacro:unless value="${simulation}">
+            <xacro:unless value="${diff_drive_emulation}">
                 <origin xyz="0.053 ${orientation * -0.043} 0.015" rpy="${orientation * M_PI/2} 0 0" />
             </xacro:unless>
@@ -93,5 +93,5 @@
             <material>Gazebo/Red</material>
         </gazebo>
-        <xacro:if value="${simulation}">
+        <xacro:if value="${diff_drive_emulation}">
             <joint name="front_wheel_${type}_joint" type="fixed">
                 <origin xyz="0 0 0" rpy="0 0 0" />

Commit message: Fix robot urdf

File: nanosaur_description/urdf/robot.urdf.xacro (robot description, xacro)
@@ -12,5 +12,6 @@
     <xacro:property name="M_PI" value="3.14159"/>
     <!--https://github.com/ros-simulation/gazebo_ros_pkgs/pull/1284 -->
-    <xacro:property name="path_meshes" value="file://$(find nanosaur_description)/meshes"/>
+    <!--I cannot use the solution below for remote machines-->
+    <!--<xacro:property name="path_meshes" value="file://$(find nanosaur_description)/meshes"/>-->
     <!--<xacro:property name="path_meshes" value="package://nanosaur_description/meshes"/>-->
     <!-- nanosaur properties -->
@@ -18,5 +19,5 @@
     <!-- Real radius 0.0105 but augmented for track thickness -->
     <xacro:property name="sprocket_radius" value="0.0150"/>
-    <xacro:macro name="nanosaur" params="cover_type use_nominal_extrinsics diff_drive_emulation">
+    <xacro:macro name="nanosaur" params="cover_type use_nominal_extrinsics diff_drive_emulation path_meshes:=package://nanosaur_description/meshes">
         <!-- Gazebo color reference
         https://bitbucket.org/osrf/gazebo/src/default/media/materials/scripts/gazebo.material?fileviewer=file-view-default

Commit message: Improve nanosaur URDF

File: nanosaur_description/urdf/robot.urdf.xacro (robot description, xacro)
@@ -21,5 +21,5 @@
     <!-- Real radius 0.0105 but augmented for track thickness -->
     <xacro:property name="sprocket_radius" value="0.0150"/>
-    <xacro:macro name="nanosaur" params="cover_type use_nominal_extrinsics diff_drive_emulation path_meshes:=package://nanosaur_description/meshes">
+    <xacro:macro name="nanosaur" params="cover_type use_nominal_extrinsics diff_drive_emulation mimic_enable:=true path_meshes:=package://nanosaur_description/meshes">
         <!-- nanosaur definition -->
         <link name="base_link" />
@@ -128,6 +128,6 @@
             </visual>
         </link>
-        <xacro:track type="left" parent="base_link" radius="${sprocket_radius}" diff_drive_emulation="${diff_drive_emulation}"/>
-        <xacro:track type="right" parent="base_link" radius="${sprocket_radius}" diff_drive_emulation="${diff_drive_emulation}"/>
+        <xacro:track type="left" parent="base_link" radius="${sprocket_radius}" diff_drive_emulation="${diff_drive_emulation}" mimic_enable="${mimic_enable}"/>
+        <xacro:track type="right" parent="base_link" radius="${sprocket_radius}" diff_drive_emulation="${diff_drive_emulation}" mimic_enable="${mimic_enable}"/>
         <xacro:flap />
         <!-- Nanosaur heads -->

File: nanosaur_description/urdf/track.urdf.xacro (robot description, xacro)
@@ -2,5 +2,5 @@
 <robot name="nanosaur_track"
     xmlns:xacro="http://ros.org/wiki/xacro">
-    <xacro:macro name="track" params="type parent radius diff_drive_emulation">
+    <xacro:macro name="track" params="type parent radius diff_drive_emulation mimic_enable">
         <!-- Define orientation -->
         <xacro:if value="${type == 'left'}">
@@ -10,4 +10,11 @@
             <xacro:property name="orientation" value="1"/>
         </xacro:if>
+        <xacro:if value="${mimic_enable}">
+            <xacro:property name="mimic_type" value="continuous"/>
+        </xacro:if>
+        <xacro:unless value="${mimic_enable}">
+            <xacro:property name="mimic_type" value="fixed"/>
+        </xacro:unless>
+        <xacro:property name="radius_wheel" value="${radius}"/>
         <joint name="sprocket_${type}_joint" type="continuous">
             <xacro:if value="${diff_drive_emulation}">
@@ -83,5 +90,5 @@
             </visual>
         </gazebo>
-        <joint name="wheel_${type}_joint" type="continuous">
+        <joint name="wheel_${type}_joint" type="${mimic_type}">
             <origin xyz="-0.099 0 0" rpy="0 0 0" />
             <parent link="motor_${type}"/>
@@ -89,5 +96,7 @@
             <axis xyz="0 0 ${-1 * orientation}" />
             <!-- Passive sprocket rotate automatically according to the status of the active one -->
-            <mimic joint="sprocket_${type}_joint" multiplier="1" offset="0"/>
+            <xacro:if value="${mimic_enable}">
+                <mimic joint="sprocket_${type}_joint" multiplier="1" offset="0"/>
+            </xacro:if>
         </joint>
         <link name="wheel_${type}">
@@ -108,5 +117,5 @@
                 <origin xyz="0 0 0" rpy="0 0 0" />
                 <geometry>
-                    <cylinder length="0.015" radius="${radius}"/>
+                    <cylinder length="0.015" radius="${radius_wheel}"/>
                 </geometry>
                 <material name="Black" />
@@ -129,10 +138,13 @@
         </gazebo>
         <xacro:if value="${diff_drive_emulation}">
-            <joint name="front_wheel_${type}_joint" type="fixed">
+            <joint name="front_wheel_${type}_joint" type="${mimic_type}">
                 <origin xyz="0 0 0" rpy="0 0 0" />
                 <parent link="motor_${type}"/>
                 <child link="front_wheel_${type}"/>
+                <axis xyz="0 0 ${-1 * orientation}" />
                 <!-- Passive sprocket rotate automatically according to the status of the active one -->
-                <mimic joint="sprocket_${type}_joint" multiplier="1" offset="0"/>
+                <xacro:if value="${mimic_enable}">
+                    <mimic joint="sprocket_${type}_joint" multiplier="1" offset="0"/>
+                </xacro:if>
             </joint>
             <link name="front_wheel_${type}">
@@ -153,5 +165,5 @@
                     <origin xyz="0 0 0" rpy="0 0 0" />
                     <geometry>
-                        <cylinder length="0.015" radius="${radius}"/>
+                        <cylinder length="0.015" radius="${radius_wheel}"/>
                     </geometry>
                     <material name="Black" />

Commit message: rename nanosaur urdf extension and fix inertia error

File: nanosaur_description/urdf/robot.urdf.xacro (robot description, xacro)
@@ -19,9 +19,9 @@
         <link name="nanosaur_base">
             <inertial>
-                <mass value="0.412"/>
+                <mass value="0.453"/>
                 <origin rpy=" 0 0 0" xyz="0.0 0 0.0"/>
-                <inertia ixx="922734.27556" ixy="0458.391" ixz="225029.72"
-                        iyy="1.701e-06" iyz="-3998.88622"
-                        izz="1995920.29749"/>
+                <inertia ixx="982653.79909" ixy="-2069.061" ixz="193876.45537"
+                        iyy="1888714.1125" iyz="-4847.17947"
+                        izz="2199329.1679"/>
             </inertial>
             <visual>
