Commit message: Improve omniwheel simulation

File: nanosaur_description/urdf/omniwheel.urdf.xacro (robot description, xacro)
@@ -13,11 +13,24 @@
         <xacro:if value="${position == 'front'}">
             <xacro:property name="motor_orientation" value="1"/>
+            <xacro:property name="fdir1_direction" value="-1"/>
         </xacro:if>
         <xacro:if value="${position == 'rear'}">
             <xacro:property name="motor_orientation" value="0"/>
+            <xacro:property name="fdir1_direction" value="1"/>
         </xacro:if>
         <!--radius definition-->
-        <xacro:property name="wheel_diameter" value="0.037"/>
-        <xacro:property name="wheel_length" value="0.0226"/>
+        <xacro:property name="omni_wheel_mass" value="0.015"/>
+        <xacro:property name="omni_wheel_radius" value="${0.037 / 2}"/>
+        <xacro:property name="omni_wheel_height" value="0.0226"/>
+        <xacro:macro name="inertial_cylinder" params="m r h">
+        <inertia  ixx="${m*(3*r*r+h*h)/12}" ixy = "0" ixz = "0"
+                    iyy="${m*r*r/2}" iyz = "0"
+                    izz="${m*(3*r*r+h*h)/12}" />
+        </xacro:macro>
+        <xacro:macro name="inertial_sphere" params="m r">
+        <inertia ixx="${(2/5) * m * (r*r)}" ixy="0.0" ixz="0.0"
+                    iyy="${(2/5) * m * (r*r)}" iyz="0.0"
+                izz="${(2/5) * m * (r*r)}" />
+        </xacro:macro>
         <joint name="motor_${type}_${position}_joint" type="fixed">
             <origin xyz="${xyz}" rpy="${orientation * M_PI/2} 0 0" />
@@ -35,17 +48,13 @@
         </link>
         <joint name="omniwheel_${type}_${position}_joint" type="continuous">
-            <origin xyz="0 0 0" rpy="0 0 0" />
+            <origin xyz="0 0 ${omni_wheel_height / 2}" rpy="0 0 0" />
             <parent link="motor_${type}_${position}"/>
             <child link="omniwheel_${type}_${position}"/>
             <axis xyz="0 0 ${-1 * orientation}" />
+            <limit effort="1000" velocity="1000"/>
         </joint>
         <link name="omniwheel_${type}_${position}">
-            <inertial>
-                <mass value="0.01"/>
-                <origin rpy=" 0 0 0" xyz="0 0 0"/>
-                <inertia ixx="1.6666666666666668e-07" ixy="0" ixz="0" iyy="1.6666666666666668e-07" iyz="0" izz="1.6666666666666668e-07"/>
-            </inertial>
             <visual>
-                <origin xyz="0 0 0" rpy="0 0 0" />
+                <origin xyz="0 0 -${omni_wheel_radius / 2}" rpy="0 0 0" />
                 <geometry>
                     <mesh filename="${path_meshes}/parts/mecanum_cover.stl"/>
@@ -55,10 +64,18 @@
             <!-- Collision cylinder -->
             <collision>
-                <origin xyz="0 0 ${wheel_length / 2}" rpy="0 0 0" />
+                <origin xyz="0 0 0" rpy="0 0 0" />
                 <geometry>
-                    <cylinder length="${wheel_length}" radius="${wheel_diameter / 2}"/>
+                    <!--<sphere radius="${omni_wheel_radius}" />-->
+                    <cylinder length="${omni_wheel_height}" radius="${omni_wheel_radius}"/>
                 </geometry>
                 <material name="Black" />
             </collision>
+            <!-- Inertia -->
+            <inertial>
+                <mass value="${omni_wheel_mass}"/>
+                <origin rpy="0 0 0" xyz="0 0 0"/>
+                <!--<xacro:inertial_sphere  m="${omni_wheel_mass}" r="${omni_wheel_radius}" />-->
+                <xacro:inertial_cylinder  m="${omni_wheel_mass}" r="${omni_wheel_radius}" h="${omni_wheel_height}" />
+            </inertial>
         </link>
         <joint name="omniwheel_${type}_${position}_wheels_joint" type="fixed">
@@ -70,5 +87,5 @@
         <link name="omniwheel_${type}_${position}_wheels">
             <visual>
-                <origin xyz="0 0 0" rpy="0 0 0" />
+                <origin xyz="0 0 -${omni_wheel_radius / 2}" rpy="0 0 0" />
                 <geometry>
                     <mesh filename="${path_meshes}/parts/mecanum_wheels.stl"/>
@@ -77,4 +94,13 @@
             </visual>
         </link>
+        <!-- Reference:
+            https://github.com/gazebosim/gz-sim/issues/2261
+        -->
+        <gazebo reference="omniwheel_${type}_${position}">
+            <mu1 value="1.0"/>
+            <mu2 value="1.0"/>
+            <fdir1 value="1 0 ${fdir1_direction}"/>
+            <turnGravityOff>false</turnGravityOff>
+        </gazebo>
     </xacro:macro>
 </robot>

Commit message: minor fixes

File: nanosaur_description/urdf/omniwheel.urdf.xacro (robot description, xacro)
@@ -51,5 +51,5 @@
             <parent link="motor_${type}_${position}"/>
             <child link="omniwheel_${type}_${position}"/>
-            <axis xyz="0 0 ${-1 * orientation}" />
+            <axis xyz="0 0 1" />
             <limit effort="1000" velocity="1000"/>
         </joint>
@@ -83,5 +83,5 @@
             <parent link="omniwheel_${type}_${position}"/>
             <child link="omniwheel_${type}_${position}_wheels"/>
-            <axis xyz="0 0 ${-1 * orientation}" />
+            <axis xyz="0 0 1" />
         </joint>
         <link name="omniwheel_${type}_${position}_wheels">
@@ -94,12 +94,8 @@
             </visual>
         </link>
-        <!-- Reference:
-            https://github.com/gazebosim/gz-sim/issues/2261
-        -->
+        <!-- Reference https://github.com/gazebosim/gz-sim/issues/2261 -->
         <gazebo reference="omniwheel_${type}_${position}">
-            <mu1 value="1.0"/>
-            <mu2 value="1.0"/>
-            <fdir1 value="1 0 ${fdir1_direction}"/>
-            <turnGravityOff>false</turnGravityOff>
+            <mu1 value="0.01"/>
+            <mu2 value="0.01"/>
         </gazebo>
     </xacro:macro>
