Commit message: Add collision for cover and minor fixes

File: nanosaur_description/urdf/head/head_fisheye.urdf.xacro (robot description, xacro)
@@ -31,4 +31,10 @@
                 <material name="Green" />
             </visual>
+            <!-- Collision cylinder -->
+            <collision>
+                <origin xyz="0.003 0 0.03" rpy="${M_PI/2} ${M_PI/2} 0" />
+                <geometry><cylinder length="0.07" radius="0.028"/></geometry>
+                <material name="Green" />
+            </collision>
         </link>
         <joint name="display_left_joint" type="fixed">

File: nanosaur_description/urdf/head/head_pi.urdf.xacro (robot description, xacro)
@@ -31,4 +31,10 @@
                 <material name="Green" />
             </visual>
+            <!-- Collision cylinder -->
+            <collision>
+                <origin xyz="-0.007 0 0.03" rpy="${M_PI/2} ${M_PI/2} 0" />
+                <geometry><cylinder length="0.07" radius="0.028"/></geometry>
+                <material name="Green" />
+            </collision>
         </link>
         <joint name="display_left_joint" type="fixed">

File: nanosaur_description/urdf/head/head_realsense.urdf.xacro (robot description, xacro)
@@ -30,4 +30,10 @@
                 <material name="Green" />
             </visual>
+            <!-- Collision cylinder -->
+            <collision>
+                <origin xyz="0.003 0 0.03" rpy="${M_PI/2} ${M_PI/2} 0" />
+                <geometry><cylinder length="0.07" radius="0.028"/></geometry>
+                <material name="Green" />
+            </collision>
         </link>
         <joint name="display_left_joint" type="fixed">

File: nanosaur_description/urdf/head/head_zedmini.urdf.xacro (robot description, xacro)
@@ -29,4 +29,10 @@
                 <material name="Green" />
             </visual>
+            <!-- Collision cylinder -->
+            <collision>
+                <origin xyz="0.003 0 0.03" rpy="${M_PI/2} ${M_PI/2} 0" />
+                <geometry><cylinder length="0.07" radius="0.028"/></geometry>
+                <material name="Green" />
+            </collision>
         </link>
         <joint name="display_left_joint" type="fixed">

File: nanosaur_description/urdf/robot.urdf.xacro (robot description, xacro)
@@ -18,5 +18,5 @@
     <xacro:macro name="nanosaur" params="cover_type use_nominal_extrinsics simulation">
         <xacro:if value="${simulation}">
-            <!-- Gazebo color reference:
+            <!-- Gazebo color reference
             https://bitbucket.org/osrf/gazebo/src/default/media/materials/scripts/gazebo.material?fileviewer=file-view-default
             http://wiki.ros.org/simulator_gazebo/Tutorials/ListOfMaterials

File: nanosaur_description/urdf/track.urdf.xacro (robot description, xacro)
@@ -2,27 +2,4 @@
 <robot name="nanosaur_track" xmlns:xacro="http://ros.org/wiki/xacro">
     <xacro:macro name="track" params="type parent radius simulation">
-        <gazebo reference="sprocket_${type}">
-            <kp>10000000</kp>
-            <kd>10000000</kd>
-            <mu1>10000000</mu1>
-            <mu2>10000000</mu2>
-            <material>Gazebo/Blue</material>
-        </gazebo>
-        <gazebo reference="motor_${type}">
-            <material>Gazebo/Gold</material>
-        </gazebo>
-        <gazebo reference="wheel_${type}">
-            <kp>10000000</kp>
-            <kd>10000000</kd>
-            <mu1>0</mu1>
-            <mu2>0</mu2>
-            <material>Gazebo/Red</material>
-        </gazebo>
-        <gazebo reference="track_${type}">
-            <material>Gazebo/Black</material>
-        </gazebo>
-        <gazebo reference="slider_${type}">
-            <material>Gazebo/Green</material>
-        </gazebo>
         <!-- Define orientation -->
         <xacro:if value="${type == 'left'}">
@@ -61,4 +38,11 @@
             </collision>
         </link>
+        <gazebo reference="sprocket_${type}">
+            <kp>10000000</kp>
+            <kd>10000000</kd>
+            <mu1>10000000</mu1>
+            <mu2>10000000</mu2>
+            <material>Gazebo/Blue</material>
+        </gazebo>
         <joint name="motor_${type}_joint" type="fixed">
             <origin xyz="0.053 ${orientation * -0.043} 0.015" rpy="${orientation * M_PI/2} 0 0" />
@@ -73,4 +57,7 @@
             </visual>
         </link>
+        <gazebo reference="motor_${type}">
+            <material>Gazebo/Gold</material>
+        </gazebo>
         <joint name="wheel_${type}_joint" type="continuous">
             <origin xyz="-0.099 0 0" rpy="0 0 0" />
@@ -99,4 +86,11 @@
             </collision>
         </link>
+        <gazebo reference="wheel_${type}">
+            <kp>10000000</kp>
+            <kd>10000000</kd>
+            <mu1>0</mu1>
+            <mu2>0</mu2>
+            <material>Gazebo/Red</material>
+        </gazebo>
         <xacro:if value="${simulation}">
             <joint name="front_wheel_${type}_joint" type="fixed">
@@ -150,4 +144,7 @@
             </visual>
         </link>
+        <gazebo reference="track_${type}">
+            <material>Gazebo/Black</material>
+        </gazebo>
         <joint name="slider_${type}_joint" type="fixed">
             <parent link="track_${type}"/>
@@ -166,4 +163,7 @@
             </visual>
         </link>
+        <gazebo reference="slider_${type}">
+            <material>Gazebo/Green</material>
+        </gazebo>
     </xacro:macro>
 </robot>
