Commit message: Fix zed model URDF name

File: nanosaur_description/urdf/head/zedmini.urdf.xacro (robot description, xacro)
@@ -1,5 +1,5 @@
 <?xml version="1.0"?>
 <robot xmlns:xacro="http://wiki.ros.org/xacro">
-  <xacro:macro name="zed_camera" params="name=zed model=zedm parent *origin">
+  <xacro:macro name="zed_camera" params="name:=zed model:=zedm parent *origin">
     <gazebo reference="${name}_camera_center">
         <material>Gazebo/Black</material>

File: nanosaur_description/urdf/robot.urdf.xacro (robot description, xacro)
@@ -162,5 +162,5 @@
         </xacro:if>
         <xacro:if value="${cover_type == 'zed'}">
-            <xacro:nanosaur_head_zedmini name="zed" />
+            <xacro:nanosaur_head_zedmini name="zedm" />
         </xacro:if>
     </xacro:macro>
