Commit message: Fix xacro for simulators

File: nanosaur_description/urdf/head/d435.urdf.xacro (robot description, xacro)
@@ -6,5 +6,6 @@
 aluminum peripherial evaluation case.
 -->
-<robot name="sensor_d435" xmlns:xacro="http://ros.org/wiki/xacro">
+<robot name="sensor_d435"
+  xmlns:xacro="http://ros.org/wiki/xacro">
   <xacro:macro name="sensor_d435" params="parent *origin name:=camera use_nominal_extrinsics:=false use_mesh:=true">
     <xacro:property name="M_PI" value="3.1415926535897931" />
@@ -40,5 +41,5 @@
     <link name="${name}_bottom_screw_frame"/>
     <joint name="${name}_link_joint" type="fixed">
-      <origin xyz="${d435_mesh_x_offset} ${d435_cam_depth_py} ${d435_cam_depth_pz}" rpy="0 0 0"/>
+      <origin xyz="-${d435_mesh_x_offset} ${d435_cam_depth_py} ${d435_cam_depth_pz}" rpy="0 0 0"/>
       <parent link="${name}_bottom_screw_frame"/>
       <child link="${name}_link" />
@@ -48,5 +49,5 @@
         <xacro:if value="${use_mesh}">
           <!-- the mesh origin is at front plate in between the two infrared camera axes -->
-          <origin xyz="${d435_zero_depth_to_glass + d435_glass_to_front} ${-d435_cam_depth_py} 0" rpy="${M_PI/2} 0 ${M_PI/2}"/>
+          <origin xyz="${d435_zero_depth_to_glass + d435_glass_to_front} ${-d435_cam_depth_py} 0" rpy="0 0 ${M_PI/2}"/>
           <geometry>
             <mesh filename="${path_meshes}/parts/d435.dae" />

File: nanosaur_description/urdf/robot.urdf.xacro (robot description, xacro)
@@ -1,5 +1,7 @@
 <?xml version="1.0"?>
 <robot name="robot" xmlns:xacro="http://ros.org/wiki/xacro">
+    <!-- materials -->
     <xacro:include filename="$(find nanosaur_description)/urdf/materials.urdf" />
+    <xacro:include filename="$(find nanosaur_description)/urdf/materials.gazebo.xacro" />
     <!-- nanosaur parts -->
     <xacro:include filename="$(find nanosaur_description)/urdf/track.urdf.xacro" />
@@ -20,9 +22,4 @@
     <xacro:property name="sprocket_radius" value="0.0150"/>
     <xacro:macro name="nanosaur" params="cover_type use_nominal_extrinsics diff_drive_emulation path_meshes:=package://nanosaur_description/meshes">
-        <!-- Gazebo color reference
-        https://bitbucket.org/osrf/gazebo/src/default/media/materials/scripts/gazebo.material?fileviewer=file-view-default
-        Gazebo http://wiki.ros.org/simulator_gazebo/Tutorials/ListOfMaterials
-        Ignition https://gazebosim.org/api/gazebo/3.7/migrationsdf.html
-        -->
         <!-- nanosaur definition -->
         <link name="base_link" />

Commit message: Update realsense mesh

File: nanosaur_description/urdf/head/d435.urdf.xacro (robot description, xacro)
@@ -41,5 +41,5 @@
     <link name="${name}_bottom_screw_frame"/>
     <joint name="${name}_link_joint" type="fixed">
-      <origin xyz="-${d435_mesh_x_offset} ${d435_cam_depth_py} ${d435_cam_depth_pz}" rpy="0 0 0"/>
+      <origin xyz="${d435_mesh_x_offset} ${d435_cam_depth_py} ${d435_cam_depth_pz}" rpy="0 0 0"/>
       <parent link="${name}_bottom_screw_frame"/>
       <child link="${name}_link" />
@@ -49,5 +49,5 @@
         <xacro:if value="${use_mesh}">
           <!-- the mesh origin is at front plate in between the two infrared camera axes -->
-          <origin xyz="${d435_zero_depth_to_glass + d435_glass_to_front} ${-d435_cam_depth_py} 0" rpy="0 0 ${M_PI/2}"/>
+          <origin xyz="${-(d435_zero_depth_to_glass + d435_glass_to_front + d435_cam_mount_from_center_offset + 0.001)} ${-d435_cam_depth_py} 0" rpy="0 0 ${M_PI/2}"/>
           <geometry>
             <mesh filename="${path_meshes}/parts/d435.dae" />
