Commit message: Improve nanosaur description and configurations

File: nanosaur_description/urdf/flap/flap.urdf.xacro (robot description, xacro)
@@ -2,18 +2,11 @@
 <robot name="nanosaur_flap"
     xmlns:xacro="http://ros.org/wiki/xacro">
-    <xacro:macro name="flap">
+    <xacro:macro name="nanosaur_flap" params="parent">
         <joint name="nanosaur_flap_joint" type="fixed">
             <origin xyz="0 0 0" rpy="0 0 0" />
-            <parent link="nanosaur_base"/>
+            <parent link="${parent}"/>
             <child link="nanosaur_flap"/>
         </joint>
         <link name="nanosaur_flap">
-            <inertial>
-                <mass value="0.018"/>
-                <origin rpy="0 0 0" xyz="-0.063 0 0.065"/>
-                <inertia ixx="7565.043" ixy="-0.00384" ixz="300.2704"
-                        iyy="2254.45646" iyz="0.00019"
-                        izz="9538.576"/>
-            </inertial>
             <visual>
                 <geometry><mesh filename="${path_meshes}/nanosaur_flap.stl" scale="0.001 0.001 0.001"/></geometry>

File: nanosaur_description/urdf/head/d435.urdf.xacro (robot description, xacro)
@@ -63,5 +63,5 @@
       </visual>
       <collision>
-        <origin xyz="0 ${-d435_cam_depth_py} 0" rpy="0 0 0"/>
+        <origin xyz="-0.008 ${-d435_cam_depth_py} 0" rpy="0 0 0"/>
         <geometry>
           <box size="${d435_cam_depth} ${d435_cam_width} ${d435_cam_height}"/>

File: nanosaur_description/urdf/omniwheel.urdf.xacro (robot description, xacro)
@@ -55,5 +55,5 @@
             <!-- Collision cylinder -->
             <collision>
-                <origin xyz="0 0 0" rpy="0 0 0" />
+                <origin xyz="0 0 ${wheel_length / 2}" rpy="0 0 0" />
                 <geometry>
                     <cylinder length="${wheel_length}" radius="${wheel_diameter / 2}"/>

File: nanosaur_description/urdf/robot.urdf.xacro (robot description, xacro)
@@ -5,6 +5,9 @@
     <xacro:include filename="$(find nanosaur_description)/urdf/materials.gazebo.xacro" />
     <!-- nanosaur parts -->
-    <xacro:include filename="$(find nanosaur_description)/urdf/flap.urdf.xacro" />
     <xacro:include filename="$(find nanosaur_description)/urdf/omniwheel.urdf.xacro" />
+    <xacro:include filename="$(find nanosaur_description)/urdf/flap/flap.urdf.xacro" />
+    <xacro:include filename="$(find nanosaur_description)/urdf/flap/flap_LD06.urdf.xacro" />
+    <xacro:include filename="$(find nanosaur_description)/urdf/head/head.urdf.xacro" />
+    <xacro:include filename="$(find nanosaur_description)/urdf/head/head_realsense.urdf.xacro" />
     <!-- Global properties -->
     <xacro:property name="M_PI" value="3.14159"/>
@@ -13,6 +16,5 @@
     <!--<xacro:property name="path_meshes" value="file://$(find nanosaur_description)/meshes"/>-->
     <!--<xacro:property name="path_meshes" value="package://nanosaur_description/meshes"/>-->
-    <!-- nanosaur properties -->
-    <xacro:macro name="nanosaur" params="cover_type use_nominal_extrinsics diff_drive_emulation mimic_enable:=true path_meshes:=package://nanosaur_description/meshes">
+    <xacro:macro name="nanosaur" params="head_type flap_type use_nominal_extrinsics diff_drive_emulation mimic_enable:=true path_meshes:=package://nanosaur_description/meshes">
         <link name="nanosaur_base">
             <inertial>
@@ -27,4 +29,11 @@
                 <material name="Green" />
             </visual>
+            <collision>
+                <origin xyz="0.01 0 0.005" rpy="0 0 0"/>
+                <geometry>
+                    <box size="0.17 0.075 0.09"/>
+                </geometry>
+                <material name="Green" />
+            </collision>
         </link>
         <joint name="nanosaur_cover_batteries_joint" type="fixed">
@@ -50,9 +59,4 @@
             </visual>
         </link>
-        <xacro:omniwheel parent="nanosaur_base" type="left" position="front" xyz="0.05 0.041 -0.035"/>
-        <xacro:omniwheel parent="nanosaur_base" type="left" position="rear" xyz="-0.05 0.041 -0.035"/>
-        <xacro:omniwheel parent="nanosaur_base" type="right" position="front" xyz="0.05 -0.041 -0.035"/>
-        <xacro:omniwheel parent="nanosaur_base" type="right" position="rear" xyz="-0.05 -0.041 -0.035"/>
-        <xacro:flap />
         <joint name="NVIDIA_jetson_joint" type="fixed">
             <origin xyz="0 0 0" rpy="0 0 0" />
@@ -141,4 +145,22 @@
             </visual>
         </link>
+        <xacro:omniwheel parent="nanosaur_base" type="left" position="front" xyz="0.05 0.041 -0.035"/>
+        <xacro:omniwheel parent="nanosaur_base" type="left" position="rear" xyz="-0.05 0.041 -0.035"/>
+        <xacro:omniwheel parent="nanosaur_base" type="right" position="front" xyz="0.05 -0.041 -0.035"/>
+        <xacro:omniwheel parent="nanosaur_base" type="right" position="rear" xyz="-0.05 -0.041 -0.035"/>
+        <!-- Nanosaur heads -->
+        <xacro:if value="${head_type == 'empty'}">
+            <xacro:nanosaur_head parent="nanosaur_base" />
+        </xacro:if>
+        <xacro:if value="${head_type == 'realsense'}">
+            <xacro:nanosaur_head_realsense parent="nanosaur_base" name="camera" use_nominal_extrinsics="${use_nominal_extrinsics}" />
+        </xacro:if>
+        <!-- Nanosaur flap -->
+        <xacro:if value="${flap_type == 'empty'}">
+            <xacro:nanosaur_flap parent="nanosaur_base" />
+        </xacro:if>
+        <xacro:if value="${flap_type == 'LD06'}">
+            <xacro:nanosaur_flap_LD06 parent="nanosaur_base" />
+        </xacro:if>
     </xacro:macro>
 </robot>
